Commit message: robot properties

File: navis_description/urdf/navis.urdf.xacro (robot description, xacro)
@@ -1 +1,6 @@
 <?xml version="1.0"?>
+  <xacro: name="wheel_radius" value="0.05"/>
+  <xacro:property name="wheel_width" value="0.02"/>
+  <xacro:property name="base_width" value="0.4"/>
+  <xacro:property name="base_length" value="0.3"/>
+  <xacro:property name="base_height" value="0.1"/>

Commit message: typo

File: navis_description/urdf/navis.urdf.xacro (robot description, xacro)
@@ -1,4 +1,4 @@
 <?xml version="1.0"?>
-  <xacro: name="wheel_radius" value="0.05"/>
+  <xacro:property name="wheel_radius" value="0.05"/>
   <xacro:property name="wheel_width" value="0.02"/>
   <xacro:property name="base_width" value="0.4"/>

Commit message: base link

File: navis_description/urdf/navis.urdf.xacro (robot description, xacro)
@@ -5,2 +5,19 @@
   <xacro:property name="base_length" value="0.3"/>
   <xacro:property name="base_height" value="0.1"/>
+  <link name="base_link">
+    <visual>
+      <geometry>
+        <box size="${base_length} ${base_width} ${base_height}"/>
+      </geometry>
+      <material name="gray"/>
+    </visual>
+    <collision>
+      <geometry>
+        <box size="${base_length} ${base_width} ${base_height}"/>
+      </geometry>
+    </collision>
+    <inertial>
+      <mass value="5.0"/>
+      <inertia ixx="0.1" iyy="0.1" izz="0.1" ixy="0.0" ixz="0.0" iyz="0.0"/>
+    </inertial>
+  </link>

Commit message: left wheel

File: navis_description/urdf/navis.urdf.xacro (robot description, xacro)
@@ -22,2 +22,11 @@
     </inertial>
   </link>
+  <!-- Left wheel -->
+  <link name="left_wheel">
+    <visual>
+      <geometry>
+        <cylinder length="${wheel_width}" radius="${wheel_radius}"/>
+      </geometry>
+      <origin xyz="0 ${base_width/2} 0" rpy="1.5708 0 0"/>
+    </visual>
+  </link>

Commit message: right wheel

File: navis_description/urdf/navis.urdf.xacro (robot description, xacro)
@@ -31,2 +31,11 @@
     </visual>
   </link>
+   <!-- Right wheel -->
+  <link name="right_wheel">
+    <visual>
+      <geometry>
+        <cylinder length="${wheel_width}" radius="${wheel_radius}"/>
+      </geometry>
+      <origin xyz="0 -${base_width/2} 0" rpy="1.5708 0 0"/>
+    </visual>
+  </link>

Commit message: back left wheel

File: navis_description/urdf/navis.urdf.xacro (robot description, xacro)
@@ -22,6 +22,6 @@
     </inertial>
   </link>
-  <!-- Left wheel -->
-  <link name="left_wheel">
+  <!-- Front Left wheel -->
+  <link name="front left_wheel">
     <visual>
       <geometry>
@@ -31,6 +31,6 @@
     </visual>
   </link>
-   <!-- Right wheel -->
-  <link name="right_wheel">
+  <!-- Front Right wheel -->
+  <link name="front right_wheel">
     <visual>
       <geometry>
@@ -40,2 +40,11 @@
     </visual>
   </link>
+  <!-- Back Left Wheel-->
+  <link name="back left_wheel">
+    <visual>
+      <geometry>
+        <cylinder length="${wheel_width}" radius="${wheel_radius}"/>
+      </geometry>
+      <origin xyz="0 ${base_width/2} 0" rpy="1.5708 0 0"/>
+    </visual>
+  </link>

Commit message: back left

File: navis_description/urdf/navis.urdf.xacro (robot description, xacro)
@@ -3,5 +3,5 @@
   <xacro:property name="wheel_width" value="0.02"/>
   <xacro:property name="base_width" value="0.4"/>
-  <xacro:property name="base_length" value="0.3"/>
+  <xacro:property name="base_length" value="0.6"/>
   <xacro:property name="base_height" value="0.1"/>
   <link name="base_link">
@@ -49,2 +49,11 @@
     </visual>
   </link>
+  <!-- Back Right wheel -->
+  <link name="back right_wheel">
+    <visual>
+      <geometry>
+        <cylinder length="${wheel_width}" radius="${wheel_radius}"/>
+      </geometry>
+      <origin xyz="0 -${base_width/2} 0" rpy="1.5708 0 0"/>
+    </visual>
+  </link>

Commit message: front left wheel joint

File: navis_description/urdf/navis.urdf.xacro (robot description, xacro)
@@ -23,5 +23,5 @@
   </link>
   <!-- Front Left wheel -->
-  <link name="front left_wheel">
+  <link name="front_left_wheel">
     <visual>
       <geometry>
@@ -32,5 +32,5 @@
   </link>
   <!-- Front Right wheel -->
-  <link name="front right_wheel">
+  <link name="front_right_wheel">
     <visual>
       <geometry>
@@ -41,5 +41,5 @@
   </link>
   <!-- Back Left Wheel-->
-  <link name="back left_wheel">
+  <link name="back_left_wheel">
     <visual>
       <geometry>
@@ -50,5 +50,5 @@
   </link>
   <!-- Back Right wheel -->
-  <link name="back right_wheel">
+  <link name="back_right_wheel">
     <visual>
       <geometry>
@@ -58,2 +58,9 @@
     </visual>
   </link>
+  <!-- Joints -->
+  <joint name"front_left_wheel_joint" type="continuous">
+    <parent link="base_link"/>
+    <child link="front_left_wheel"/>
+    <origin xyz="0 ${base_width/2} 0"/ rpy="0 0 0">
+    <axis xyz="0 0 1"/>
+  </joint>

Commit message: front right wheel joint

File: navis_description/urdf/navis.urdf.xacro (robot description, xacro)
@@ -65,2 +65,8 @@
     <axis xyz="0 0 1"/>
   </joint>
+  <joint name="front_right_wheel_joint" type="continuous">
+    <parent link="base_link"/>
+    <child link="front_right_wheel"/>
+    <origin xyz="0 -${base_width/2} 0" rpy="0 0 0"/>
+    <axis xyz="0 0 1"/>
+  </joint>

Commit message: back wheel joints

File: navis_description/urdf/navis.urdf.xacro (robot description, xacro)
@@ -71,2 +71,14 @@
     <axis xyz="0 0 1"/>
   </joint>
+  <joint name"back_left_wheel_joint" type="continuous">
+    <parent link="base_link"/>
+    <child link="back_left_wheel"/>
+    <origin xyz="0 ${base_width/2} 0"/ rpy="0 0 0">
+    <axis xyz="0 0 1"/>
+  </joint>
+  <joint name"back_right_wheel_joint" type="continuous">
+    <parent link="base_link"/>
+    <child link="back_right_wheel"/>
+    <origin xyz="0 ${base_width/2} 0"/ rpy="0 0 0">
+    <axis xyz="0 0 1"/>
+  </joint>

Commit message: depth camera

File: navis_description/urdf/navis.urdf.xacro (robot description, xacro)
@@ -83,2 +83,11 @@
     <axis xyz="0 0 1"/>
   </joint>
+  <!-- Depth Camera -->
+  <link name="depth_camera_link">
+    <visual>
+      <geometry>
+        <box size="0.05 0.05 0.05"/>
+      </geometry>
+      <origin xyz="0.1 0 0.1"/>
+    </visual>
+  </link>

Commit message: depth camera lnk + comments

File: navis_description/urdf/navis.urdf.xacro (robot description, xacro)
@@ -1,3 +1,4 @@
 <?xml version="1.0"?>
+  <!-- Properties -->
   <xacro:property name="wheel_radius" value="0.05"/>
   <xacro:property name="wheel_width" value="0.02"/>
@@ -5,4 +6,5 @@
   <xacro:property name="base_length" value="0.6"/>
   <xacro:property name="base_height" value="0.1"/>
+  <!-- Base Link -->
   <link name="base_link">
     <visual>
@@ -58,5 +60,5 @@
     </visual>
   </link>
-  <!-- Joints -->
+  <!-- Wheel Joints -->
   <joint name"front_left_wheel_joint" type="continuous">
     <parent link="base_link"/>
@@ -92,2 +94,7 @@
     </visual>
   </link>
+  <joint name="depth_camera_joint" type="fixed">
+    <parent link="base_link"/>
+    <child link="depth_camera_link"/>
+    <origin xyz="0.1 0 0.1" rpy="0 0 0"/>
+  </joint>

Commit message: added mesh property

File: navis_description/urdf/navis.urdf.xacro (robot description, xacro)
@@ -2,4 +2,5 @@
 <robot xmlns:xacro="http://ros.org/wiki/xacro" name="navis">
   <!-- Properties -->
+  <xacro:property name="chassis_mesh" value="package://navis_description/meshes/x2_chassis.dae"/>
   <xacro:property name="wheel_radius" value="0.05"/>
   <xacro:property name="wheel_width" value="0.02"/>

Commit message: simplified urdf

File: navis_description/urdf/navis.urdf.xacro (robot description, xacro)
@@ -3,101 +3,29 @@
   <!-- Properties -->
   <xacro:property name="chassis_mesh" value="package://navis_description/meshes/x2_chassis.dae"/>
-  <xacro:property name="wheel_radius" value="0.05"/>
-  <xacro:property name="wheel_width" value="0.02"/>
-  <xacro:property name="base_width" value="0.4"/>
-  <xacro:property name="base_length" value="0.6"/>
-  <xacro:property name="base_height" value="0.1"/>
-  <!-- Base Link -->
+  <xacro:property name="chassis_mass" value="20.0"/> <!-- in kg -->
+  <xacro:property name="chassis_size_x" value="0.6"/>
+  <xacro:property name="chassis_size_y" value="0.5"/>
+  <xacro:property name="chassis_size_z" value="0.25"/>
   <link name="base_link">
     <visual>
+      <origin xyz="0 0 0" rpy="0 0 0"/>
       <geometry>
-        <box size="${base_length} ${base_width} ${base_height}"/>
+        <mesh filename="${chassis_mesh}" scale="1 1 1"/>
       </geometry>
-      <material name="gray"/>
     </visual>
     <collision>
+      <origin xyz="0 0 0" rpy="0 0 0"/>
       <geometry>
-        <box size="${base_length} ${base_width} ${base_height}"/>
+        <box size="${chassis_size_x} ${chassis_size_y} ${chassis_size_z}"/>
       </geometry>
     </collision>
     <inertial>
-      <mass value="5.0"/>
-      <inertia ixx="0.1" iyy="0.1" izz="0.1" ixy="0.0" ixz="0.0" iyz="0.0"/>
+      <mass value="${chassis_mass}"/>
+      <origin xyz="0 0 0" rpy="0 0 0"/>
+      <inertia
+        ixx="1.0" ixy="0.0" ixz="0.0"
+        iyy="1.0" iyz="0.0"
+        izz="1.0"/>
     </inertial>
   </link>
-  <!-- Front Left wheel -->
-  <link name="front_left_wheel">
-    <visual>
-      <geometry>
-        <cylinder length="${wheel_width}" radius="${wheel_radius}"/>
-      </geometry>
-      <origin xyz="0 ${base_width/2} 0" rpy="1.5708 0 0"/>
-    </visual>
-  </link>
-  <!-- Front Right wheel -->
-  <link name="front_right_wheel">
-    <visual>
-      <geometry>
-        <cylinder length="${wheel_width}" radius="${wheel_radius}"/>
-      </geometry>
-      <origin xyz="0 -${base_width/2} 0" rpy="1.5708 0 0"/>
-    </visual>
-  </link>
-  <!-- Back Left Wheel-->
-  <link name="back_left_wheel">
-    <visual>
-      <geometry>
-        <cylinder length="${wheel_width}" radius="${wheel_radius}"/>
-      </geometry>
-      <origin xyz="0 ${base_width/2} 0" rpy="1.5708 0 0"/>
-    </visual>
-  </link>
-  <!-- Back Right wheel -->
-  <link name="back_right_wheel">
-    <visual>
-      <geometry>
-        <cylinder length="${wheel_width}" radius="${wheel_radius}"/>
-      </geometry>
-      <origin xyz="0 -${base_width/2} 0" rpy="1.5708 0 0"/>
-    </visual>
-  </link>
-  <!-- Wheel Joints -->
-  <joint name"front_left_wheel_joint" type="continuous">
-    <parent link="base_link"/>
-    <child link="front_left_wheel"/>
-    <origin xyz="0 ${base_width/2} 0"/ rpy="0 0 0">
-    <axis xyz="0 0 1"/>
-  </joint>
-  <joint name="front_right_wheel_joint" type="continuous">
-    <parent link="base_link"/>
-    <child link="front_right_wheel"/>
-    <origin xyz="0 -${base_width/2} 0" rpy="0 0 0"/>
-    <axis xyz="0 0 1"/>
-  </joint>
-  <joint name"back_left_wheel_joint" type="continuous">
-    <parent link="base_link"/>
-    <child link="back_left_wheel"/>
-    <origin xyz="0 ${base_width/2} 0"/ rpy="0 0 0">
-    <axis xyz="0 0 1"/>
-  </joint>
-  <joint name"back_right_wheel_joint" type="continuous">
-    <parent link="base_link"/>
-    <child link="back_right_wheel"/>
-    <origin xyz="0 ${base_width/2} 0"/ rpy="0 0 0">
-    <axis xyz="0 0 1"/>
-  </joint>
-  <!-- Depth Camera -->
-  <link name="depth_camera_link">
-    <visual>
-      <geometry>
-        <box size="0.05 0.05 0.05"/>
-      </geometry>
-      <origin xyz="0.1 0 0.1"/>
-    </visual>
-  </link>
-  <joint name="depth_camera_joint" type="fixed">
-    <parent link="base_link"/>
-    <child link="depth_camera_link"/>
-    <origin xyz="0.1 0 0.1" rpy="0 0 0"/>
-  </joint>
 </robot>

Commit message: robot urdf update

File: navis_description/urdf/navis.urdf.xacro (robot description, xacro)
@@ -1,31 +1,128 @@
 <?xml version="1.0"?>
-<robot xmlns:xacro="http://ros.org/wiki/xacro" name="navis">
-  <!-- Properties -->
-  <xacro:property name="chassis_mesh" value="package://navis_description/meshes/x2_chassis.dae"/>
-  <xacro:property name="chassis_mass" value="20.0"/> <!-- in kg -->
-  <xacro:property name="chassis_size_x" value="0.6"/>
-  <xacro:property name="chassis_size_y" value="0.5"/>
-  <xacro:property name="chassis_size_z" value="0.25"/>
+<robot xmlns:xacro="http://www.ros.org/wiki/xacro" name="navis">
+  <!-- Base parameters -->
+  <xacro:property name="base_length" value="0.42" />
+  <xacro:property name="base_width" value="0.31" />
+  <xacro:property name="base_height" value="0.184" />
+  <xacro:property name="base_mass" value="16.524" />
+  <xacro:property name="wheel_radius" value="0.098" />
+  <xacro:property name="wheel_length" value="0.04" />
+  <xacro:property name="wheel_mass" value="0.477" />
+  <!-- Base link -->
   <link name="base_link">
-    <visual>
-      <origin xyz="0 0 0" rpy="0 0 0"/>
+    <inertial>
+      <origin xyz="0.011999 0.002 0.066996" rpy="0 0 0"/>
+      <mass value="${base_mass}"/>
+      <inertia
+        ixx="0.320605" ixy="-0.000800023" ixz="0.0163992"
+        iyy="0.399205" iyz="-0.000900133"
+        izz="0.455501"/>
+    </inertial>
+    <collision name="chassis_collision">
+      <origin xyz="0 0 0.092" rpy="0 0 0"/>
       <geometry>
-        <mesh filename="${chassis_mesh}" scale="1 1 1"/>
+        <box size="${base_length} ${base_width} ${base_height}"/>
+      </geometry>
+    </collision>
+    <visual name="chassis_visual">
+      <origin xyz="0 0 -0.0655" rpy="1.5708 0 -1.5708"/>
+      <geometry>
+        <mesh filename="package://X2/meshes/x2_chassis.dae"/>
       </geometry>
     </visual>
-    <collision>
-      <origin xyz="0 0 0" rpy="0 0 0"/>
+    <!-- Sensors -->
+    <xacro:include filename="$(find X2)/urdf/sensors.xacro"/>
+    <xacro:imu_sensor parent="base_link"
+      xyz="0 0 0" rpy="0 0 0"
+      noise_mean="0" noise_stddev="0.007"/>
+    <xacro:stereo_camera parent="base_link"
+      left_xyz="0.23 0.1 0.19" left_rpy="0 0 0"
+      right_xyz="0.23 -0.1 0.19" right_rpy="0 0 0"
+      width="1280" height="960" hfov="1.0472"/>
+    <!-- Visual elements -->
+    <visual name="navsat_visual_1">
+      <origin xyz="-0.18 0.126 0.1895" rpy="0 0 0"/>
       <geometry>
-        <box size="${chassis_size_x} ${chassis_size_y} ${chassis_size_z}"/>
+        <cylinder length="0.016" radius="0.026"/>
       </geometry>
-    </collision>
-    <inertial>
-      <mass value="${chassis_mass}"/>
-      <origin xyz="0 0 0" rpy="0 0 0"/>
-      <inertia
-        ixx="1.0" ixy="0.0" ixz="0.0"
-        iyy="1.0" iyz="0.0"
-        izz="1.0"/>
-    </inertial>
+    </visual>
+    <!-- Headlights -->
+    <xacro:macro name="headlight" params="name xyz rpy">
+      <visual name="${name}">
+        <origin xyz="${xyz}" rpy="${rpy}"/>
+        <geometry>
+          <mesh filename="package://X2/meshes/headlight.dae"/>
+        </geometry>
+      </visual>
+    </xacro:macro>
+    <xacro:headlight name="center_left_headlight_visual"
+      xyz="0.22 0.05 0.0845" rpy="0 0 -3.14159"/>
+    <xacro:headlight name="left_headlight_visual"
+      xyz="0.22 0.145 0.0845" rpy="0 0 -3.14159"/>
+    <xacro:headlight name="center_right_headlight_visual"
+      xyz="0.22 -0.05 0.0845" rpy="0 0 -3.14159"/>
+    <xacro:headlight name="right_headlight_visual"
+      xyz="0.22 -0.145 0.0845" rpy="0 0 -3.14159"/>
   </link>
+  <!-- Wheel macro -->
+  <xacro:macro name="wheel" params="prefix xyz reflect">
+    <link name="${prefix}_wheel">
+      <inertial>
+        <mass value="${wheel_mass}"/>
+        <inertia
+          ixx="0.0013" ixy="0" ixz="0"
+          iyy="0.0024" iyz="0"
+          izz="0.0013"/>
+      </inertial>
+      <collision name="${prefix}_collision">
+        <origin xyz="0 0 0" rpy="1.5708 0 0"/>
+        <geometry>
+          <cylinder radius="${wheel_radius}" length="${wheel_length}"/>
+        </geometry>
+        <surface>
+          <friction>
+            <ode mu="1" mu2="1" slip1="0.0026" slip2="0"/>
+          </friction>
+        </surface>
+      </collision>
+      <visual name="${prefix}_visual">
+        <origin xyz="0 0 0" rpy="1.5708 0 0"/>
+        <geometry>
+          <mesh filename="package://X2/meshes/x2_wheel_${'left' if reflect > 0 else 'right'}.dae"/>
+        </geometry>
+      </visual>
+    </link>
+    <joint name="${prefix}_wheel_joint" type="continuous">
+      <parent link="base_link"/>
+      <child link="${prefix}_wheel"/>
+      <origin xyz="${xyz}" rpy="0 0 0"/>
+      <axis xyz="0 1 0"/>
+    </joint>
+    <transmission name="${prefix}_wheel_trans">
+      <type>transmission_interface/SimpleTransmission</type>
+      <joint name="${prefix}_wheel_joint">
+        <hardwareInterface>hardware_interface/VelocityJointInterface</hardwareInterface>
+      </joint>
+      <actuator name="${prefix}_wheel_motor">
+        <hardwareInterface>hardware_interface/VelocityJointInterface</hardwareInterface>
+        <mechanicalReduction>1</mechanicalReduction>
+      </actuator>
+    </transmission>
+  </xacro:macro>
+  <!-- Create wheels -->
+  <xacro:wheel prefix="front_left" xyz="0.131 0.187795 0.0345" reflect="1"/>
+  <xacro:wheel prefix="front_right" xyz="0.131 -0.187795 0.0345" reflect="-1"/>
+  <xacro:wheel prefix="rear_left" xyz="-0.131 0.187795 0.0345" reflect="1"/>
+  <xacro:wheel prefix="rear_right" xyz="-0.131 -0.187795 0.0345" reflect="-1"/>
+  <!-- Gazebo extensions -->
+  <gazebo>
+    <plugin name="gazebo_ros_control" filename="libgazebo_ros_control.so">
+      <robotNamespace>/X2</robotNamespace>
+    </plugin>
+  </gazebo>
+  <gazebo reference="base_link">
+    <mu1>0.2</mu1>
+    <mu2>0.2</mu2>
+    <material>Gazebo/Grey</material>
+  </gazebo>
 </robot>
