Commit message: imu macro

File: navis_description/urdf/robots/navis.urdf.xacro (robot description, xacro)
@@ -32,5 +32,27 @@
     </visual>
     <!-- IMU -->
-    <xacro:navis_imu parent="base_link"/>
+    <!-- <xacro:navis_imu parent="base_link"/> -->
+    <xacro:macro name="navis_imu" params="">
+      <link name="imu_link">
+        <visual>
+          <geometry>
+            <box size="0.05 0.05 0.02"/>
+          </geometry>
+          <material name="gray"/>
+        </visual>
+        <inertial>
+          <mass value="0.01"/>
+          <origin xyz="0 0 0" rpy="0 0 0"/>
+          <inertia ixx="0.0001" ixy="0.0" ixz="0.0"
+                  iyy="0.0001" iyz="0.0"
+                  izz="0.0001"/>
+        </inertial>
+      </link>
+      <joint name="imu_joint" type="fixed">
+        <parent link="base_link"/>
+        <child link="imu_link"/>
+        <origin xyz="0 0 0.1" rpy="0 0 0"/>
+      </joint>
+    </xacro:macro>
     <!-- Visual elements -->
     <visual name="navsat_visual_1">

Commit message: update urdf

File: navis_description/urdf/robots/navis.urdf.xacro (robot description, xacro)
@@ -31,4 +31,5 @@
       </geometry>
     </visual>
+  </link>
     <!-- IMU -->
     <!-- <xacro:navis_imu parent="base_link"/> -->

Commit message: comment out navsat_visual

File: navis_description/urdf/robots/navis.urdf.xacro (robot description, xacro)
@@ -33,5 +33,5 @@
   </link>
     <!-- IMU -->
-    <!-- <xacro:navis_imu parent="base_link"/> -->
+    <xacro:navis_imu parent="base_link"/>
     <xacro:macro name="navis_imu" params="">
       <link name="imu_link">
@@ -57,10 +57,10 @@
     </xacro:macro>
     <!-- Visual elements -->
-    <visual name="navsat_visual_1">
+    <!-- <visual name="navsat_visual_1">
       <origin xyz="-0.18 0.126 0.1895" rpy="0 0 0"/>
       <geometry>
         <cylinder length="0.016" radius="0.026"/>
       </geometry>
-    </visual>
+    </visual> -->
     <!-- Headlights -->
     <xacro:macro name="headlight" params="name xyz rpy">

Commit message: add world link

File: navis_description/urdf/robots/navis.urdf.xacro (robot description, xacro)
@@ -142,3 +142,8 @@
     <material>Gazebo/Grey</material>
   </gazebo>
+  <link name="world"/>
+    <joint name="world_joint" type="fixed">
+      <parent link="world"/>
+      <child link="base_link"/>
+    </joint>
 </robot>

Commit message: add world origin

File: navis_description/urdf/robots/navis.urdf.xacro (robot description, xacro)
@@ -146,4 +146,5 @@
       <parent link="world"/>
       <child link="base_link"/>
+       <origin xyz="0 0 0" rpy="0 0 0"/>
     </joint>
 </robot>

Commit message: fix file paths

File: navis_description/urdf/robots/navis.urdf.xacro (robot description, xacro)
@@ -29,5 +29,5 @@
       <origin xyz="0 0 -0.0655" rpy="1.5708 0 -1.5708"/>
       <geometry>
-        <mesh filename="package://X2/meshes/x2_chassis.dae"/>
+        <mesh filename="package://navis_description/meshes/x2_chassis.dae"/>
       </geometry>
     </visual>
@@ -69,5 +69,5 @@
         <origin xyz="${xyz}" rpy="${rpy}"/>
         <geometry>
-          <mesh filename="package://X2/meshes/headlight.dae"/>
+          <mesh filename="package://navis_description/meshes/headlight.dae"/>
         </geometry>
       </visual>
@@ -106,5 +106,5 @@
         <origin xyz="0 0 0" rpy="1.5708 0 0"/>
         <geometry>
-          <mesh filename="package://X2/meshes/x2_wheel_${'left' if reflect > 0 else 'right'}.dae"/>
+          <mesh filename="package://navis_description/meshes/x2_wheel_${'left' if reflect > 0 else 'right'}.dae"/>
         </geometry>
       </visual>

Commit message: comment out mesh paths

File: navis_description/urdf/robots/navis.urdf.xacro (robot description, xacro)
@@ -29,5 +29,6 @@
       <origin xyz="0 0 -0.0655" rpy="1.5708 0 -1.5708"/>
       <geometry>
-        <mesh filename="package://navis_description/meshes/x2_chassis.dae"/>
+        <!-- <mesh filename="package://navis_description/meshes/x2_chassis.dae"/> -->
+        <box size="0.2 0.2 0.2"/>
       </geometry>
     </visual>
@@ -69,5 +70,6 @@
         <origin xyz="${xyz}" rpy="${rpy}"/>
         <geometry>
-          <mesh filename="package://navis_description/meshes/headlight.dae"/>
+          <!-- <mesh filename="package://navis_description/meshes/headlight.dae"/> -->
+          <box size="0.2 0.2 0.2"/>
         </geometry>
       </visual>
@@ -106,5 +108,6 @@
         <origin xyz="0 0 0" rpy="1.5708 0 0"/>
         <geometry>
-          <mesh filename="package://navis_description/meshes/x2_wheel_${'left' if reflect > 0 else 'right'}.dae"/>
+          <!-- <mesh filename="package://navis_description/meshes/x2_wheel_${'left' if reflect > 0 else 'right'}.dae"/> -->
+          <box size="0.2 0.2 0.2"/>
         </geometry>
       </visual>

Commit message: comment out entire code

File: navis_description/urdf/robots/navis.urdf.xacro (robot description, xacro)
@@ -1,6 +1,6 @@
-<?xml version="1.0"?>
+<!-- <?xml version="1.0"?>
 <robot xmlns:xacro="http://www.ros.org/wiki/xacro" name="navis">
   <xacro:include filename="$navis_descripiton/urdf/sensors/imu.urdf.xacro" />
-  <!-- Base parameters -->
+  Base parameters
   <xacro:property name="base_length" value="0.42" />
   <xacro:property name="base_width" value="0.31" />
@@ -10,5 +10,5 @@
   <xacro:property name="wheel_length" value="0.04" />
   <xacro:property name="wheel_mass" value="0.477" />
-  <!-- Base link -->
+  Base link
   <link name="base_link">
     <inertial>
@@ -29,10 +29,10 @@
       <origin xyz="0 0 -0.0655" rpy="1.5708 0 -1.5708"/>
       <geometry>
-        <!-- <mesh filename="package://navis_description/meshes/x2_chassis.dae"/> -->
+        <mesh filename="package://navis_description/meshes/x2_chassis.dae"/>
         <box size="0.2 0.2 0.2"/>
       </geometry>
     </visual>
   </link>
-    <!-- IMU -->
+    IMU
     <xacro:navis_imu parent="base_link"/>
     <xacro:macro name="navis_imu" params="">
@@ -58,6 +58,6 @@
       </joint>
     </xacro:macro>
-    <!-- Visual elements -->
-    <!-- <visual name="navsat_visual_1">
+    Visual elements
+    <visual name="navsat_visual_1">
       <origin xyz="-0.18 0.126 0.1895" rpy="0 0 0"/>
       <geometry>
@@ -65,10 +65,10 @@
       </geometry>
     </visual> -->
-    <!-- Headlights -->
+    <!-- Headlights
     <xacro:macro name="headlight" params="name xyz rpy">
       <visual name="${name}">
         <origin xyz="${xyz}" rpy="${rpy}"/>
         <geometry>
-          <!-- <mesh filename="package://navis_description/meshes/headlight.dae"/> -->
+          <mesh filename="package://navis_description/meshes/headlight.dae"/>
           <box size="0.2 0.2 0.2"/>
         </geometry>
@@ -84,5 +84,5 @@
       xyz="0.22 -0.145 0.0845" rpy="0 0 -3.14159"/>
   </link>
-  <!-- Wheel macro -->
+  Wheel macro
   <xacro:macro name="wheel" params="prefix xyz reflect">
     <link name="${prefix}_wheel">
@@ -108,5 +108,5 @@
         <origin xyz="0 0 0" rpy="1.5708 0 0"/>
         <geometry>
-          <!-- <mesh filename="package://navis_description/meshes/x2_wheel_${'left' if reflect > 0 else 'right'}.dae"/> -->
+          <mesh filename="package://navis_description/meshes/x2_wheel_${'left' if reflect > 0 else 'right'}.dae"/>
           <box size="0.2 0.2 0.2"/>
         </geometry>
@@ -130,10 +130,10 @@
     </transmission>
   </xacro:macro>
-  <!-- Create wheels -->
+  Create wheels
   <xacro:wheel prefix="front_left" xyz="0.131 0.187795 0.0345" reflect="1"/>
   <xacro:wheel prefix="front_right" xyz="0.131 -0.187795 0.0345" reflect="-1"/>
   <xacro:wheel prefix="rear_left" xyz="-0.131 0.187795 0.0345" reflect="1"/>
   <xacro:wheel prefix="rear_right" xyz="-0.131 -0.187795 0.0345" reflect="-1"/>
-  <!-- Gazebo extensions -->
+  Gazebo extensions
   <gazebo>
     <plugin name="gazebo_ros_control" filename="libgazebo_ros_control.so">
@@ -152,3 +152,3 @@
        <origin xyz="0 0 0" rpy="0 0 0"/>
     </joint>
-</robot>
+</robot> -->

Commit message: basic xacro for test

File: navis_description/urdf/robots/navis.urdf.xacro (robot description, xacro)
@@ -1,2 +1,31 @@
+<?xml version="1.0"?>
+<robot xmlns:xacro="http://www.ros.org/wiki/xacro" name="navis">
+  <!-- Simple base link with a box -->
+  <link name="base_link">
+    <visual>
+      <origin xyz="0 0 0.1" rpy="0 0 0"/>
+      <geometry>
+        <box size="0.5 0.3 0.2"/>
+      </geometry>
+      <material name="green">
+        <color rgba="0 1.0 0 1.0"/>
+      </material>
+    </visual>
+    <collision>
+      <origin xyz="0 0 0.1" rpy="0 0 0"/>
+      <geometry>
+        <box size="0.5 0.3 0.2"/>
+      </geometry>
+    </collision>
+    <inertial>
+      <mass value="1.0"/>
+      <origin xyz="0 0 0.1" rpy="0 0 0"/>
+      <inertia
+        ixx="0.1" ixy="0.0" ixz="0.0"
+        iyy="0.1" iyz="0.0"
+        izz="0.1"/>
+    </inertial>
+  </link>
+</robot>
 <!-- <?xml version="1.0"?>
 <robot xmlns:xacro="http://www.ros.org/wiki/xacro" name="navis">

Commit message: ulstra simple model for test

File: navis_description/urdf/robots/navis.urdf.xacro (robot description, xacro)
@@ -1,29 +1,10 @@
 <?xml version="1.0"?>
 <robot xmlns:xacro="http://www.ros.org/wiki/xacro" name="navis">
-  <!-- Simple base link with a box -->
   <link name="base_link">
     <visual>
-      <origin xyz="0 0 0.1" rpy="0 0 0"/>
       <geometry>
-        <box size="0.5 0.3 0.2"/>
+        <box size="0.2 0.2 0.1"/>
       </geometry>
-      <material name="green">
-        <color rgba="0 1.0 0 1.0"/>
-      </material>
     </visual>
-    <collision>
-      <origin xyz="0 0 0.1" rpy="0 0 0"/>
-      <geometry>
-        <box size="0.5 0.3 0.2"/>
-      </geometry>
-    </collision>
-    <inertial>
-      <mass value="1.0"/>
-      <origin xyz="0 0 0.1" rpy="0 0 0"/>
-      <inertia
-        ixx="0.1" ixy="0.0" ixz="0.0"
-        iyy="0.1" iyz="0.0"
-        izz="0.1"/>
-    </inertial>
   </link>
 </robot>

Commit message: minimal model test cube

File: navis_description/urdf/robots/navis.urdf.xacro (robot description, xacro)
@@ -1,8 +1,8 @@
 <?xml version="1.0"?>
-<robot xmlns:xacro="http://www.ros.org/wiki/xacro" name="navis">
+<robot xmlns:xacro="http://ros.org/wiki/xacro" name="navis">
   <link name="base_link">
     <visual>
       <geometry>
-        <box size="0.2 0.2 0.1"/>
+        <box size="0.3 0.3 0.3"/>
       </geometry>
     </visual>

Commit message: urdf simplification

File: navis_description/urdf/robots/navis.urdf.xacro (robot description, xacro)
@@ -1,164 +1,5 @@
 <?xml version="1.0"?>
-<robot xmlns:xacro="http://ros.org/wiki/xacro" name="navis">
-  <link name="base_link">
-    <visual>
-      <geometry>
-        <box size="0.3 0.3 0.3"/>
-      </geometry>
-    </visual>
-  </link>
-</robot>
-<!-- <?xml version="1.0"?>
 <robot xmlns:xacro="http://www.ros.org/wiki/xacro" name="navis">
   <xacro:include filename="$navis_descripiton/urdf/sensors/imu.urdf.xacro" />
-  Base parameters
-  <xacro:property name="base_length" value="0.42" />
-  <xacro:property name="base_width" value="0.31" />
-  <xacro:property name="base_height" value="0.184" />
-  <xacro:property name="base_mass" value="16.524" />
-  <xacro:property name="wheel_radius" value="0.098" />
-  <xacro:property name="wheel_length" value="0.04" />
-  <xacro:property name="wheel_mass" value="0.477" />
-  Base link
-  <link name="base_link">
-    <inertial>
-      <origin xyz="0.011999 0.002 0.066996" rpy="0 0 0"/>
-      <mass value="${base_mass}"/>
-      <inertia
-        ixx="0.320605" ixy="-0.000800023" ixz="0.0163992"
-        iyy="0.399205" iyz="-0.000900133"
-        izz="0.455501"/>
-    </inertial>
-    <collision name="chassis_collision">
-      <origin xyz="0 0 0.092" rpy="0 0 0"/>
-      <geometry>
-        <box size="${base_length} ${base_width} ${base_height}"/>
-      </geometry>
-    </collision>
-    <visual name="chassis_visual">
-      <origin xyz="0 0 -0.0655" rpy="1.5708 0 -1.5708"/>
-      <geometry>
-        <mesh filename="package://navis_description/meshes/x2_chassis.dae"/>
-        <box size="0.2 0.2 0.2"/>
-      </geometry>
-    </visual>
-  </link>
-    IMU
-    <xacro:navis_imu parent="base_link"/>
-    <xacro:macro name="navis_imu" params="">
-      <link name="imu_link">
-        <visual>
-          <geometry>
-            <box size="0.05 0.05 0.02"/>
-          </geometry>
-          <material name="gray"/>
-        </visual>
-        <inertial>
-          <mass value="0.01"/>
-          <origin xyz="0 0 0" rpy="0 0 0"/>
-          <inertia ixx="0.0001" ixy="0.0" ixz="0.0"
-                  iyy="0.0001" iyz="0.0"
-                  izz="0.0001"/>
-        </inertial>
-      </link>
-      <joint name="imu_joint" type="fixed">
-        <parent link="base_link"/>
-        <child link="imu_link"/>
-        <origin xyz="0 0 0.1" rpy="0 0 0"/>
-      </joint>
-    </xacro:macro>
-    Visual elements
-    <visual name="navsat_visual_1">
-      <origin xyz="-0.18 0.126 0.1895" rpy="0 0 0"/>
-      <geometry>
-        <cylinder length="0.016" radius="0.026"/>
-      </geometry>
-    </visual> -->
-    <!-- Headlights
-    <xacro:macro name="headlight" params="name xyz rpy">
-      <visual name="${name}">
-        <origin xyz="${xyz}" rpy="${rpy}"/>
-        <geometry>
-          <mesh filename="package://navis_description/meshes/headlight.dae"/>
-          <box size="0.2 0.2 0.2"/>
-        </geometry>
-      </visual>
-    </xacro:macro>
-    <xacro:headlight name="center_left_headlight_visual"
-      xyz="0.22 0.05 0.0845" rpy="0 0 -3.14159"/>
-    <xacro:headlight name="left_headlight_visual"
-      xyz="0.22 0.145 0.0845" rpy="0 0 -3.14159"/>
-    <xacro:headlight name="center_right_headlight_visual"
-      xyz="0.22 -0.05 0.0845" rpy="0 0 -3.14159"/>
-    <xacro:headlight name="right_headlight_visual"
-      xyz="0.22 -0.145 0.0845" rpy="0 0 -3.14159"/>
-  </link>
-  Wheel macro
-  <xacro:macro name="wheel" params="prefix xyz reflect">
-    <link name="${prefix}_wheel">
-      <inertial>
-        <mass value="${wheel_mass}"/>
-        <inertia
-          ixx="0.0013" ixy="0" ixz="0"
-          iyy="0.0024" iyz="0"
-          izz="0.0013"/>
-      </inertial>
-      <collision name="${prefix}_collision">
-        <origin xyz="0 0 0" rpy="1.5708 0 0"/>
-        <geometry>
-          <cylinder radius="${wheel_radius}" length="${wheel_length}"/>
-        </geometry>
-        <surface>
-          <friction>
-            <ode mu="1" mu2="1" slip1="0.0026" slip2="0"/>
-          </friction>
-        </surface>
-      </collision>
-      <visual name="${prefix}_visual">
-        <origin xyz="0 0 0" rpy="1.5708 0 0"/>
-        <geometry>
-          <mesh filename="package://navis_description/meshes/x2_wheel_${'left' if reflect > 0 else 'right'}.dae"/>
-          <box size="0.2 0.2 0.2"/>
-        </geometry>
-      </visual>
-    </link>
-    <joint name="${prefix}_wheel_joint" type="continuous">
-      <parent link="base_link"/>
-      <child link="${prefix}_wheel"/>
-      <origin xyz="${xyz}" rpy="0 0 0"/>
-      <axis xyz="0 1 0"/>
-    </joint>
-    <transmission name="${prefix}_wheel_trans">
-      <type>transmission_interface/SimpleTransmission</type>
-      <joint name="${prefix}_wheel_joint">
-        <hardwareInterface>hardware_interface/VelocityJointInterface</hardwareInterface>
-      </joint>
-      <actuator name="${prefix}_wheel_motor">
-        <hardwareInterface>hardware_interface/VelocityJointInterface</hardwareInterface>
-        <mechanicalReduction>1</mechanicalReduction>
-      </actuator>
-    </transmission>
-  </xacro:macro>
-  Create wheels
-  <xacro:wheel prefix="front_left" xyz="0.131 0.187795 0.0345" reflect="1"/>
-  <xacro:wheel prefix="front_right" xyz="0.131 -0.187795 0.0345" reflect="-1"/>
-  <xacro:wheel prefix="rear_left" xyz="-0.131 0.187795 0.0345" reflect="1"/>
-  <xacro:wheel prefix="rear_right" xyz="-0.131 -0.187795 0.0345" reflect="-1"/>
-  Gazebo extensions
-  <gazebo>
-    <plugin name="gazebo_ros_control" filename="libgazebo_ros_control.so">
-      <robotNamespace>/X2</robotNamespace>
-    </plugin>
-  </gazebo>
-  <gazebo reference="base_link">
-    <mu1>0.2</mu1>
-    <mu2>0.2</mu2>
-    <material>Gazebo/Grey</material>
-  </gazebo>
-  <link name="world"/>
-    <joint name="world_joint" type="fixed">
-      <parent link="world"/>
-      <child link="base_link"/>
-       <origin xyz="0 0 0" rpy="0 0 0"/>
-    </joint>
-</robot> -->
+<link name="world"></link>
+</robot>

Commit message: base joint

File: navis_description/urdf/robots/navis.urdf.xacro (robot description, xacro)
@@ -1,4 +1,10 @@
 <?xml version="1.0"?>
 <robot xmlns:xacro="http://www.ros.org/wiki/xacro" name="navis">
+  <!-- World link -->
 <link name="world"></link>
+<joint name="base_joint" type="fixed">
+    <origin xyz="1.5 1.0 0" rpy="0 0 0"/>
+    <parent link="world"/>
+    <child link="base_link"/>
+</joint>
 </robot>

Commit message: base link name

File: navis_description/urdf/robots/navis.urdf.xacro (robot description, xacro)
@@ -10,3 +10,5 @@
 </joint>
 <!-- base link-->
+<link name="base_link">
+</link>
 </robot>

Commit message: base link

File: navis_description/urdf/robots/navis.urdf.xacro (robot description, xacro)
@@ -11,4 +11,10 @@
 <!-- base link-->
 <link name="base_link">
+    <visual>
+        <origin xyz="0 0 0.05" rpy="0 0 0"/>
+        <geometry>
+            <cylinder height>
+        </geometry>
+    </visual>
 </link>
 </robot>

Commit message: base link

File: navis_description/urdf/robots/navis.urdf.xacro (robot description, xacro)
@@ -9,3 +9,6 @@
     <child link="base_link"/>
 </joint>
+<!-- base link-->
+<link name="base_link">
+</link>
 </robot>
